Commit message: forgot to replace car with flipkart

File: models/realsense/realsense-RS200.macro.xacro (robot description, xacro)
@@ -17,5 +17,5 @@
             <origin rpy="0 0 0" xyz="0 0 0"/>
             <geometry>
-                <mesh filename="package://car/urdf/sensors/realsense/meshes/realsense.dae"/>
+                <mesh filename="package://flipkart/models/realsense/meshes/realsense.dae"/>
             </geometry>
         </visual>
