Commit message: changes

File: Flipkart_Files/bumblebee_depth_camera/bumblebee_depth_camera.urdf (robot description, URDF)
Before this commit: robot bumblebee_depth_camera, 11 links, 10 joints
Links:
- link base_link: geometry collision box size=0.47 0.47 0.11; visual mesh filename=package://rotors_gazebo/models/rotors_description/meshes/bu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 scale=0.001 0.001 0.001

File: models/bumblebee_depth_camera/bumblebee_depth_camera.urdf (robot description, URDF)
Before this commit: robot bumblebee_depth_camera, 11 links, 10 joints
Links:
- link base_link: geometry collision box size=0.47 0.47 0.11; visual mesh filename=package://flipkart/models/meshes/bumblebee.stl scale=0.001 0.001 0.001
- link depth_camera_link: geometry visual mesh filename=package://flipkart/models/meshes/realsense.dae scale=1.0 1.0 1.0
- link rotor_0: geometry collision cylinder length=0.005 radius=0.128; visual mesh filename=package://flipkart/models/meshes/iris_prop_ccw.dae scale=1 1 1
- link rotor_1: geometry collision cylinder length=0.005 radius=0.128; visual mesh filename=package://flipkart/models/meshes/iris_prop_ccw.dae scale=1 1 1
- link rotor_2: geometry collision cylinder length=0.005 radius=0.128; visual mesh filename=package://flipkart/models/meshes/iris_prop_cw.dae scale=1 1 1
- link rotor_3: geometry collision cylinder length=0.005 radius=0.128; visual mesh filename=package://flipkart/models/meshes/iris_prop_cw.dae scale=1 1 1
- link rotor_4: geometry collision cylinder length=0.005 radius=0.128; visual mesh filename=package://flipkart/models/meshes/iris_prop_cw.dae scale=1 1 1
- link rotor_5: geometry collision cylinder length=0.005 radius=0.128; visual mesh filename=package://flipkart/models/meshes/iris_prop_cw.dae scale=1 1 1
- link rotor_6: geometry collision cylinder length=0.005 radius=0.128; visual mesh filename=package://flipkart/models/meshes/iris_prop_ccw.dae scale=1 1 1
- link rotor_7: geometry collision cylinder length=0.005 radius=0.128; visual mesh filename=package://flipkart/models/meshes/iris_prop_ccw.dae scale=1 1 1
