Commit message: changes 1

File: models/bumblebee_depth_camera/bumblebee_depth_camera.urdf (robot description, URDF)
Before this commit: robot bumblebee_depth_camera, 11 links, 10 joints
Links:
- link depth_camera_link: geometry visual mesh filename=package://flipkart/models/realsense_camera/meshes/realsense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 scale=1.0 1.0 1.0
